Commit message: Single robot appears to work fine

File: create_description/urdf/create.urdf (robot description, URDF)
Before this commit: robot create, 3 links, 2 joints
Joints:
- removed joint left_wheel
- removed joint right_wheel
- added joint left_wheel_joint: type continuous, parent base, child left_wheel, axis 0 1 0
- added joint right_wheel_joint: type continuous, parent base, child right_wheel, axis 0 1 0
