Commit message: Add configurable namespace

File: create_description/urdf/create.urdf.xacro (robot description, xacro)
@@ -28,16 +28,18 @@
       </geometry>
       <gazebo>
-      <surface>
-	      <friction>
-	      <ode>
-            <mu>0</mu>
-            <mu2>0</mu2>
-            <fdir1>0 0 0</fdir1>
-            <slip1>0</slip1>
-            <slip2>0</slip2>
-          </ode>
-        </friction>
-      </surface>
-    </gazebo>
+        <surface>
+          <friction>
+            <ode>
+              <mu>0</mu>
+              <mu2>0</mu2>
+              <fdir1>0 0 0</fdir1>
+              <slip1>0</slip1>
+              <slip2>0</slip2>
+            </ode>
+          </friction>
+        </surface>
+        <mu>0</mu>
+        <mu2>0</mu2>
+      </gazebo>
     </collision>
     <visual name="front_wheel_visual">
@@ -53,15 +55,19 @@
         <sphere radius="0.015000"/>
       </geometry>
-      <surface>
-        <friction>
-          <ode>
-            <mu>0</mu>
-            <mu2>0</mu2>
-            <fdir1>0 0 0</fdir1>
-            <slip1>0</slip1>
-            <slip2>0</slip2>
-          </ode>
-        </friction>
-      </surface>
+      <gazebo>
+        <surface>
+          <friction>
+            <ode>
+              <mu>0</mu>
+              <mu2>0</mu2>
+              <fdir1>0 0 0</fdir1>
+              <slip1>0</slip1>
+              <slip2>0</slip2>
+            </ode>
+          </friction>
+        </surface>
+        <mu>0</mu>
+        <mu2>0</mu2>
+      </gazebo>
     </collision>
     <visual name="rear_wheel_visual">
@@ -164,14 +170,15 @@
   </link>
   <link name="left_wheel">
-    <origin xyz="0 0.130000 0.032000" rpy="0 0 0"/>
     <inertial>
+      <origin xyz="0 0.130000 0.032000" rpy="0 0 0"/>
       <inertia ixx="0.001000" ixy="0" ixz="0" iyy="0.001000" iyz="0" izz="0.001000"/>
       <mass value="0.010000"/>
     </inertial>
     <collision name="collision">
-      <origin xyz="0 0 0" rpy="0 1.570700 1.570700"/>
-      <geometry>
-        <cylinder radius="0.033000" length="0.023000"/>
-      </geometry>
+      <origin xyz="0 0.13 0.032" rpy="0 1.570700 1.570700"/>
+      <geometry>
+        <cylinder radius="0.033000" length="0.023000"/>
+      </geometry>
+      <gazebo>
       <surface>
         <friction>
@@ -185,7 +192,10 @@
         </friction>
       </surface>
+      <mu>10</mu>
+      <mu2>10</mu2>
+    </gazebo>
     </collision>
     <visual name="visual">
-      <origin xyz="0 0 0" rpy="0 1.570700 1.570700"/>
+      <origin xyz="0 0.13 0.032" rpy="0 1.570700 1.570700"/>
       <geometry>
         <cylinder radius="0.033000" length="0.023000"/>
@@ -194,14 +204,15 @@
   </link>
   <link name="right_wheel">
-    <origin xyz="0 -0.130000 0.032000" rpy="0 0 0"/>
     <inertial>
+      <origin xyz="0 -0.130000 0.032000" rpy="0 0 0"/>
       <inertia ixx="0.001000" ixy="0" ixz="0" iyy="0.001000" iyz="0" izz="0.001000"/>
       <mass value="0.010000"/>
     </inertial>
     <collision name="collision">
-      <origin xyz="0 0 0" rpy="0 1.570700 1.570700"/>
-      <geometry>
-        <cylinder radius="0.033000" length="0.023000"/>
-      </geometry>
+      <origin xyz="0 -0.13 0.032" rpy="0 1.570700 1.570700"/>
+      <geometry>
+        <cylinder radius="0.033000" length="0.023000"/>
+      </geometry>
+      <gazebo>
       <surface>
         <friction>
@@ -215,7 +226,10 @@
         </friction>
       </surface>
+      <mu>10</mu>
+      <mu2>10</mu2>
+    </gazebo>
     </collision>
     <visual name="visual">
-      <origin xyz="0 0 0" rpy="0 1.570700 1.570700"/>
+      <origin xyz="0 -0.13 0.032" rpy="0 1.570700 1.570700"/>
       <geometry>
         <cylinder radius="0.033000" length="0.023000"/>
@@ -223,10 +237,10 @@
     </visual>
   </link>
-  <joint name="left_wheel" type="continuous">
+  <joint name="left_wheel_joint" type="continuous">
     <parent link="base"/>
     <child link="left_wheel"/>
     <axis xyz="0 1 0"/>
   </joint>
-  <joint name="right_wheel" type="continuous">
+  <joint name="right_wheel_joint" type="continuous">
     <parent link="base"/>
     <child link="right_wheel"/>
@@ -238,5 +252,5 @@
       <mechanicalReduction>1</mechanicalReduction>
     </actuator>
-    <joint name="left_wheel">
+    <joint name="left_wheel_joint">
       <hardwareInterface>VelocityJointInterface</hardwareInterface>
     </joint>
@@ -247,7 +261,12 @@
       <mechanicalReduction>1</mechanicalReduction>
     </actuator>
-    <joint name="right_wheel">
+    <joint name="right_wheel_joint">
       <hardwareInterface>VelocityJointInterface</hardwareInterface>
     </joint>
   </transmission>
+  <gazebo>
+    <plugin name="gazebo_ros_control" filename="libgazebo_ros_control.so">
+      <robotNamespace>/$(arg namespace)</robotNamespace>
+    </plugin>
+  </gazebo>
 </robot>

Commit message: Debugging the URDF

File: create_description/urdf/create.urdf.xacro (robot description, xacro)
@@ -13,5 +13,5 @@
       <origin xyz="0 0 0.047800" rpy="0 0 0"/>
       <geometry>
-        <cylinder radius="0.016495" length="0.061163"/>
+        <cylinder radius="0.16495" length="0.061163"/>
       </geometry>
     </collision>
@@ -27,19 +27,4 @@
         <sphere radius="0.018000"/>
       </geometry>
-      <gazebo>
-        <surface>
-          <friction>
-            <ode>
-              <mu>0</mu>
-              <mu2>0</mu2>
-              <fdir1>0 0 0</fdir1>
-              <slip1>0</slip1>
-              <slip2>0</slip2>
-            </ode>
-          </friction>
-        </surface>
-        <mu>0</mu>
-        <mu2>0</mu2>
-      </gazebo>
     </collision>
     <visual name="front_wheel_visual">
@@ -55,19 +40,4 @@
         <sphere radius="0.015000"/>
       </geometry>
-      <gazebo>
-        <surface>
-          <friction>
-            <ode>
-              <mu>0</mu>
-              <mu2>0</mu2>
-              <fdir1>0 0 0</fdir1>
-              <slip1>0</slip1>
-              <slip2>0</slip2>
-            </ode>
-          </friction>
-        </surface>
-        <mu>0</mu>
-        <mu2>0</mu2>
-      </gazebo>
     </collision>
     <visual name="rear_wheel_visual">
@@ -180,19 +150,4 @@
         <cylinder radius="0.033000" length="0.023000"/>
       </geometry>
-      <gazebo>
-      <surface>
-        <friction>
-          <ode>
-            <mu>10</mu>
-            <mu2>10</mu2>
-            <fdir1>0 0 0</fdir1>
-            <slip1>0</slip1>
-            <slip2>0</slip2>
-          </ode>
-        </friction>
-      </surface>
-      <mu>10</mu>
-      <mu2>10</mu2>
-    </gazebo>
     </collision>
     <visual name="visual">
@@ -214,19 +169,4 @@
         <cylinder radius="0.033000" length="0.023000"/>
       </geometry>
-      <gazebo>
-      <surface>
-        <friction>
-          <ode>
-            <mu>10</mu>
-            <mu2>10</mu2>
-            <fdir1>0 0 0</fdir1>
-            <slip1>0</slip1>
-            <slip2>0</slip2>
-          </ode>
-        </friction>
-      </surface>
-      <mu>10</mu>
-      <mu2>10</mu2>
-    </gazebo>
     </collision>
     <visual name="visual">
@@ -270,3 +210,15 @@
     </plugin>
   </gazebo>
+  <gazebo reference="base">
+    <mu1>0</mu1>
+    <mu2>0</mu2>
+  </gazebo>
+  <gazebo reference="left_wheel">
+    <mu1>10</mu1>
+    <mu2>10</mu2>
+  </gazebo>
+  <gazebo reference="right_wheel">
+    <mu1>10</mu1>
+    <mu2>10</mu2>
+  </gazebo>
 </robot>

Commit message: Fix transforms

File: create_description/urdf/create.urdf.xacro (robot description, xacro)
@@ -141,10 +141,10 @@
   <link name="left_wheel">
     <inertial>
-      <origin xyz="0 0.130000 0.032000" rpy="0 0 0"/>
+      <origin xyz="0 0 0" rpy="0 0 0"/>
       <inertia ixx="0.001000" ixy="0" ixz="0" iyy="0.001000" iyz="0" izz="0.001000"/>
       <mass value="0.010000"/>
     </inertial>
     <collision name="collision">
-      <origin xyz="0 0.13 0.032" rpy="0 1.570700 1.570700"/>
+      <origin xyz="0 0 0" rpy="0 1.570700 1.570700"/>
       <geometry>
         <cylinder radius="0.033000" length="0.023000"/>
@@ -152,5 +152,5 @@
     </collision>
     <visual name="visual">
-      <origin xyz="0 0.13 0.032" rpy="0 1.570700 1.570700"/>
+      <origin xyz="0 0 0" rpy="0 1.570700 1.570700"/>
       <geometry>
         <cylinder radius="0.033000" length="0.023000"/>
@@ -160,10 +160,10 @@
   <link name="right_wheel">
     <inertial>
-      <origin xyz="0 -0.130000 0.032000" rpy="0 0 0"/>
+      <origin xyz="0 0 0" rpy="0 0 0"/>
       <inertia ixx="0.001000" ixy="0" ixz="0" iyy="0.001000" iyz="0" izz="0.001000"/>
       <mass value="0.010000"/>
     </inertial>
     <collision name="collision">
-      <origin xyz="0 -0.13 0.032" rpy="0 1.570700 1.570700"/>
+      <origin xyz="0 0 0" rpy="0 1.570700 1.570700"/>
       <geometry>
         <cylinder radius="0.033000" length="0.023000"/>
@@ -171,5 +171,5 @@
     </collision>
     <visual name="visual">
-      <origin xyz="0 -0.13 0.032" rpy="0 1.570700 1.570700"/>
+      <origin xyz="0 0 0" rpy="0 1.570700 1.570700"/>
       <geometry>
         <cylinder radius="0.033000" length="0.023000"/>
@@ -178,4 +178,5 @@
   </link>
   <joint name="left_wheel_joint" type="continuous">
+    <origin xyz="0 0.13 0.032" rpy="0 0 0"/>
     <parent link="base"/>
     <child link="left_wheel"/>
@@ -183,4 +184,5 @@
   </joint>
   <joint name="right_wheel_joint" type="continuous">
+    <origin xyz="0 -0.13 0.032" rpy="0 0 0"/>
     <parent link="base"/>
     <child link="right_wheel"/>

Commit message: Minor launch file updates

File: create_description/urdf/create.urdf.xacro (robot description, xacro)
@@ -16,4 +16,15 @@
       </geometry>
     </collision>
+    <collision name="contact_sensor">
+      <origin xyz="0 0 0.047800" rpy="0 0 0"/>
+      <geometry>
+        <cylinder radius="0.16495" length="0.061163"/>
+      </geometry>
+    </collision>
+    <sensor name='my_sensor' type='contact'>
+      <contact>
+        <collision>contact_sensr</collision>
+      </contact>
+    </sensor>
     <visual name="base_visual">
       <origin xyz="0 0 0.047800" rpy="0 0 0"/>
